Commit message: modell got very unstable as soon as steering was introduced while driving, got much better with significantly higher p values, tested increasing d with very bad results. keep d low

File: src/bobcat_description/urdf/bobcat.xacro (robot description, xacro)
@@ -39,5 +39,5 @@
   </link>
   <joint name="left_rear_wheel_joint" type="continuous">
-    <origin xyz="0 0.1 0" rpy="1.5708 0 0" />
+    <origin xyz="0 0.11 0" rpy="1.5708 0 0" />
     <parent link="chassis" />
     <child link="left_rear_wheel" />
@@ -60,5 +60,5 @@
   </link>
   <joint name="right_rear_wheel_joint" type="continuous">
-    <origin xyz="0 -0.1 0" rpy="1.5708 0 0" />
+    <origin xyz="0 -0.11 0" rpy="1.5708 0 0" />
     <parent link="chassis" />
     <child link="right_rear_wheel" />
@@ -78,5 +78,5 @@
   </link>
   <joint name="left_steering_hinge_joint" type="revolute">
-    <origin xyz="0.325 0.1 0" rpy="0 1.5708 0" />
+    <origin xyz="0.325 0.11 0" rpy="0 1.5708 0" />
     <parent link="chassis" />
     <child link="left_steering_hinge" />
@@ -96,5 +96,5 @@
   </link>
   <joint name="right_steering_hinge_joint" type="revolute">
-    <origin xyz="0.325 -0.1 0" rpy="0 1.5708 0" />
+    <origin xyz="0.325 -0.11 0" rpy="0 1.5708 0" />
     <parent link="chassis" />
     <child link="right_steering_hinge" />

Commit message: first changes made long way to go. This commit is done before changing chassis with base_link

File: src/bobcat_description/urdf/bobcat.xacro (robot description, xacro)
@@ -2,11 +2,55 @@
 <robot name="racecar" xmlns:xacro="http://www.ros.org/wiki/xacro">
   <xacro:include filename="$(find bobcat_description)/urdf/macros.xacro" />
+  <xacro:property name="PI" value="3.1415926835897931"/>
+<!--  <xacro:property name="base_height" value="0"/> -->
+  <xacro:property name="base_height" value="1.0639"/>
+  <xacro:property name="base_mass" value="2050"/>
+  <xacro:property name="base_mass_ixx" value="63"/>
+  <xacro:property name="base_mass_iyy" value="1048"/>
+  <xacro:property name="base_mass_izz" value="1111"/>
+  <xacro:property name="base_mass_ixz" value="-31"/>
+  <xacro:property name="tyre_x" value="1.31"/>
+  <xacro:property name="tyre_y" value="0.765"/>
+  <xacro:property name="tyre_length" value="0.229"/>
+  <xacro:property name="tyre_r" value="0.66"/>
+  <xacro:property name="tyre_radius" value="0.356"/>
+  <xacro:property name="tyre_mass" value="40"/>
+  <xacro:property name="tyre_mass_ixx" value="54"/>
+  <xacro:property name="tyre_mass_iyy" value="56"/>
+  <xacro:property name="tyre_mass_izz" value="104"/>
+  <xacro:property name="car_height" value="0.8"/>
+  <xacro:property name="car_width" value="1.440"/>
+  <xacro:property name="car_length" value="1.54"/>
+  <xacro:property name="camera_box" value="0.1"/>
+  <xacro:property name="tyre_height" value="-0.696"/>
+  <xacro:property name="str_length" value="0.01"/>
+  <xacro:property name="str_radius" value="0.1"/>
+  <xacro:property name="str_angle" value="0.6"/>
+  <xacro:property name="tyre_origin">
+	<origin xyz="0 0 0" rpy="${PI/2} 0 0"/>
+  </xacro:property>
+  <xacro:property name="tyre_origin_2">
+        <origin xyz="0 0 0" rpy="0 0 ${PI/2}"/>
+  </xacro:property>
+  <xacro:property name="tyre_origin_3">
+        <origin xyz="0 0 0" rpy="0 0 ${-PI/2}"/>
+  </xacro:property>
   <!-- Add chassis and it's inertia link -->
   <link name="base_link" />
   <link name="chassis">
     <visual>
-      <xacro:chassis_geometry/>
+      <!--xacro:chassis_geometry/-->
+      <origin xyz="0 0 0" rpy="0 0 0" />
+      <geometry>
+        <box size="${car_length} ${car_width} ${car_height}"/>
+      </geometry>
       <material name="blue" />
     </visual>
+    <collision>
+	<origin xyz="0 0 ${base_height}" rpy= "0 0 0"/>
+        <geometry>
+            <box size="${car_length} ${car_width} ${car_height}"/>
+        </geometry>
+    </collision>
   </link>
   <joint name="base_link_joint" type="fixed">
@@ -17,6 +61,12 @@
   <link name="chassis_inertia">
     <inertial>
-      <xacro:chassis_inertial_params />
-    </inertial>
+      <!--xacro:chassis_inertial_params /-->
+      <origin xyz="0 0 ${base_height}" rpy="0 0 0" />
+      <mass value="${base_mass}" />
+      <inertia
+          ixx="${base_mass_ixx}"  ixy="0.000000" ixz="${base_mass_ixz}"
+          iyy="${base_mass_iyy}" iyz="0.000000"
+          izz="${base_mass_izz}"/>
+      </inertial>
   </link>
   <joint name="chassis_inertia_joint" type="fixed">
@@ -43,5 +93,5 @@
     <child link="left_rear_wheel" />
     <axis xyz="0 0 -1" />
-    <limit effort="10" velocity="100" />
+    <limit effort="10000" velocity="100" />
   </joint>
   <xacro:wheel_transmission name="left_rear_wheel" />

File: src/bobcat_description/urdf/macros.xacro (robot description, xacro)
@@ -48,5 +48,6 @@
   <origin xyz="0 0 0" rpy="0 0 0" />
   <geometry>
-    <mesh filename="package://bobcat_description/meshes/chassis.STL" />
+    <!--mesh filename="package://bobcat_description/meshes/chassis.STL" /-->
+    <box size="${car_length} ${car_width} ${car_height}"/>
   </geometry>
 </xacro:macro>

Commit message: was time to make a new commit most of the new model is already looking pretty good havent tested the controllers

File: src/bobcat_description/urdf/bobcat.xacro (robot description, xacro)
@@ -13,4 +13,5 @@
   <xacro:property name="tyre_y" value="0.765"/>
   <xacro:property name="tyre_length" value="0.229"/>
+  <xacro:property name="tyre_height" value="-0.696"/>
   <xacro:property name="tyre_r" value="0.66"/>
   <xacro:property name="tyre_radius" value="0.356"/>
@@ -20,8 +21,7 @@
   <xacro:property name="tyre_mass_izz" value="104"/>
   <xacro:property name="car_height" value="0.8"/>
-  <xacro:property name="car_width" value="1.440"/>
-  <xacro:property name="car_length" value="1.54"/>
+  <xacro:property name="car_width" value="1.301"/>
+  <xacro:property name="car_length" value="2.62"/>
   <xacro:property name="camera_box" value="0.1"/>
-  <xacro:property name="tyre_height" value="-0.696"/>
   <xacro:property name="str_length" value="0.01"/>
   <xacro:property name="str_radius" value="0.1"/>
@@ -37,14 +37,5 @@
   </xacro:property>
   <!-- Add chassis and it's inertia link -->
-  <link name="base_link" />
-  <link name="chassis">
-    <visual>
-      <!--xacro:chassis_geometry/-->
-      <origin xyz="0 0 0" rpy="0 0 0" />
-      <geometry>
-        <box size="${car_length} ${car_width} ${car_height}"/>
-      </geometry>
-      <material name="blue" />
-    </visual>
+  <link name="base_link">
     <collision>
 	<origin xyz="0 0 ${base_height}" rpy= "0 0 0"/>
@@ -53,11 +44,14 @@
         </geometry>
     </collision>
-  </link>
-  <joint name="base_link_joint" type="fixed">
-    <origin xyz="0 0 0.05" rpy="0 0 0" />
-    <parent link="base_link" />
-    <child link="chassis" />
-  </joint>
-  <link name="chassis_inertia">
+    <visual>
+      <!--xacro:chassis_geometry/-->
+      <origin xyz="0 0 ${base_height}" rpy="0 0 0" />
+      <geometry>
+        <box size="${car_length} ${car_width} ${car_height}"/>
+      </geometry>
+      <material name="blue" />
+    </visual>
+  </link>
+  <link name="main_mass">
     <inertial>
       <!--xacro:chassis_inertial_params /-->
@@ -66,135 +60,233 @@
       <inertia
           ixx="${base_mass_ixx}"  ixy="0.000000" ixz="${base_mass_ixz}"
-          iyy="${base_mass_iyy}" iyz="0.000000"
+          iyy="${base_mass_iyy}"  iyz="0.000000"
           izz="${base_mass_izz}"/>
       </inertial>
   </link>
-  <joint name="chassis_inertia_joint" type="fixed">
+  <joint name="inertia_joint" type="fixed">
+    <parent link="base_link" />
+    <child link="main_mass" />
     <origin xyz="0 0 0" rpy="0 0 0" />
-    <parent link="chassis" />
-    <child link="chassis_inertia" />
-  </joint>
-  <!-- Add the left rear wheel with its joints and tranmissions -->
+  </joint>
+  <!-- Left Rear Wheel -->
   <link name="left_rear_wheel">
-    <inertial>
-      <xacro:left_wheels_inertial_params />
-    </inertial>
-    <visual>
-      <xacro:left_rear_wheel_geometry />
+    <collision>
+      <xacro:insert_block name="tyre_origin"/>
+      <!--xacro:left_wheels_collision_geometry/-->
+      <geometry>
+        <cylinder length="${tyre_length}" radius="${tyre_radius}"/>
+      </geometry>
+    </collision>
+    <visual>
+      <!--xacro:left_rear_wheel_geometry /-->
+      <xacro:insert_block name="tyre_origin"/>
+      <geometry>
+        <cylinder length="${tyre_length}" radius="${tyre_radius}"/>
+      </geometry>
       <material name="black" />
     </visual>
-    <collision>robot
-      <xacro:left_wheels_collision_geometry />
-    </collision>
+    <inertial>
+      <!--xacro:left_wheels_inertial_params /-->
+      <origin xyz="0 0 0" rpy="0 0 0"/>
+      <mass value="${tyre_mass}"/>
+      <inertia
+          ixx="${tyre_mass_ixx}"  ixy="0.000000"  ixz="0.000000"
+          iyy="${tyre_mass_iyy}"  iyz="0.000000"
+          izz="${tyre_mass_izz}"/>
+    </inertial>
   </link>
   <joint name="left_rear_wheel_joint" type="continuous">
-    <origin xyz="0 0.11 0" rpy="1.5708 0 0" />
-    <parent link="chassis" />
+    <parent link="base_link" />
     <child link="left_rear_wheel" />
-    <axis xyz="0 0 -1" />
+    <origin xyz="${-tyre_x} ${tyre_y} ${tyre_r}" rpy="0 0 0"/>
+    <axis xyz="0 1 0" />
+    <dynamics damping="0.1"/>
     <limit effort="10000" velocity="100" />
-  </joint>
+    <joint_properties damping="0.0" friction="0.0" />
+  </joint>
+  <!-- this transmission is added to connect to wheel effort controller! dont delete"-->
   <xacro:wheel_transmission name="left_rear_wheel" />
-  <!-- Add the right rear wheel with its joints and tranmissions -->
+  <!-- Right Rear Wheel -->
   <link name="right_rear_wheel">
-    <inertial>
-      <xacro:right_wheels_inertial_params />
-    </inertial>
-    <visual>
-      <xacro:right_rear_wheel_geometry />
+    <collision>
+      <!--xacro:right_wheels_collision_geometry /-->
+      <xacro:insert_block name="tyre_origin"/>
+      <geometry>
+        <cylinder length="${tyre_length}" radius="${tyre_radius}"/>
+      </geometry>
+    </collision>
+    <visual>
+      <xacro:insert_block name="tyre_origin"/>
+      <!--xacro:right_rear_wheel_geometry /-->
+      <geometry>
+        <cylinder length="${tyre_length}" radius="${tyre_radius}"/>
+      </geometry>
       <material name="black" />
     </visual>
-    <collision>
-      <xacro:right_wheels_collision_geometry />
-    </collision>
+    <inertial>
+      <!--xacro:right_wheels_inertial_params /-->
+      <origin xyz="0 0 0" rpy="0 0 0"/>
+      <mass value="${tyre_mass}"/>
+      <inertia
+          ixx="${tyre_mass_ixx}"  ixy="0.000000"  ixz="0.000000"
+          iyy="${tyre_mass_iyy}"  iyz="0.000000"
+          izz="${tyre_mass_izz}"/>
+    </inertial>
   </link>
   <joint name="right_rear_wheel_joint" type="continuous">
-    <origin xyz="0 -0.11 0" rpy="1.5708 0 0" />
-    <parent link="chassis" />
+    <parent link="base_link" />
     <child link="right_rear_wheel" />
-    <axis xyz="0 0 -1" />
-    <limit effort="10" velocity="100" />
-  </joint>
+    <origin xyz="${-tyre_x} ${-tyre_y} ${tyre_r}" rpy="0 0 0"/>
+    <axis xyz="0 1 0"/>
+    <dynamics damping="0.1"/>
+    <limit effort="10000" velocity="100" />
+    <joint_properties damping="0.0" friction="0.0" />
+  </joint>
+  <!-- this transmission is added to connect to wheel effort controller! dont delete"-->
   <xacro:wheel_transmission name="right_rear_wheel" />
-  <!-- Add the left steering hinge with its joints and tranmissions -->
+  <!-- Left Steering Hinge -->
   <link name="left_steering_hinge">
-    <inertial>
-      <xacro:steering_hinge_inertial_params />
-    </inertial>
-    <visual>
-      <xacro:left_steering_hinge_geometry />
+    <collision>
+      <xacro:insert_block name="tyre_origin"/>
+      <geometry>
+        <cylinder length="${str_length}" radius="${str_radius}"/>
+      </geometry>
+    </collision>
+    <visual>
+      <!--xacro:left_steering_hinge_geometry /-->
+      <xacro:insert_block name="tyre_origin"/>
+      <geometry>
+        <cylinder length="${str_length}" radius="${str_radius}"/>
+      </geometry>
       <material name="grey" />
     </visual>
+      <inertial>
+        <origin xyz="0 0 0" rpy="0 0 0"/>
+        <mass value="10.00"/>
+        <inertia
+          ixx="0.4"  ixy="0.000000"  ixz="0.000000"
+          iyy="0.6"  iyz="0.000000"
+          izz="0.4"/>
+    </inertial>
   </link>
   <joint name="left_steering_hinge_joint" type="revolute">
-    <origin xyz="0.325 0.11 0" rpy="0 1.5708 0" />
-    <parent link="chassis" />
+    <parent link="base_link" />
     <child link="left_steering_hinge" />
-    <axis xyz="-1 0 0" />
-    <limit lower="-0.5" upper="0.5" effort="1" velocity="1" />
-  </joint>
+    <origin xyz="${tyre_x} ${car_width/2 + str_length/2} ${tyre_r}" rpy="0 0 0"/>
+    <axis xyz="0 0 1"/>
+    <limit effort="1000.0" lower="${-str_angle}" upper="${str_angle}" velocity="0.5"/>
+  </joint>
+  <!-- this transmission is added to connect to wheel effort controller! dont delete"-->
   <xacro:steering_hinge_transmission name="left_steering_hinge" />
-  <!-- Add the right steering hinge with its joints and tranmissions -->
+  <!-- Right Steering Hinge -->
   <link name="right_steering_hinge">
-    <inertial>
-      <xacro:steering_hinge_inertial_params />
-    </inertial>
-    <visual>
-      <xacro:right_steering_hinge_geometry />
-      <material name="grey" />
-    </visual>
+    <collision>
+      <xacro:insert_block name="tyre_origin"/>
+      <geometry>
+        <cylinder length="${tyre_length}" radius="${tyre_radius}"/>
+      </geometry>
+    </collision>
+    <visual>
+      <xacro:insert_block name="tyre_origin"/>
+      <geometry>
+        <cylinder length="${str_length}" radius="${str_radius}"/>
+      </geometry>
+    </visual>
+    <inertial>
+      <origin xyz="0 0 0" rpy="0 0 0"/>
+      <mass value="10.00"/>
+      <inertia
+          ixx="0.4"  ixy="0.000000"  ixz="0.000000"
+          iyy="0.6"  iyz="0.000000"
+          izz="0.4"/>
+    </inertial>
   </link>
   <joint name="right_steering_hinge_joint" type="revolute">
-    <origin xyz="0.325 -0.11 0" rpy="0 1.5708 0" />
-    <parent link="chassis" />
+    <parent link="base_link" />
     <child link="right_steering_hinge" />
-    <axis xyz="-1 0 0" />
-    <limit lower="-0.5" upper="0.5" effort="1" velocity="1" />
-  </joint>
+    <origin xyz="${tyre_x} ${-car_width/2 - str_length/2} ${tyre_r}" rpy="0 0 0"/>
+    <axis xyz="0 0 1"/>
+    <limit effort="1000.0" lower="${-str_angle}" upper="${str_angle}" velocity="0.5"/>
+  </joint>
+  <!-- this transmission is added to connect to wheel effort controller! dont delete"-->
   <xacro:steering_hinge_transmission name="right_steering_hinge" />
-  <!-- Add the left front wheel with its joints and tranmissions -->
+  <!-- Left Front Wheel -->
   <link name="left_front_wheel">
-    <inertial>
-      <xacro:left_wheels_inertial_params />
-    </inertial>
-    <visual>
-      <xacro:left_front_wheel_geometry />
+    <collision>
+      <!--xacro:left_wheels_collision_geometry /-->
+      <xacro:insert_block name="tyre_origin"/>
+      <geometry>
+         <cylinder length="${tyre_length}" radius="${tyre_radius}"/>
+      </geometry>
+    </collision>
+    <visual>
+      <!--xacro:left_front_wheel_geometry /-->
+      <xacro:insert_block name="tyre_origin"/>
+      <geometry>
+         <cylinder length="${tyre_length}" radius="${tyre_radius}"/>
+      </geometry>
       <material name="black" />
     </visual>
-    <collision>
-      <xacro:left_wheels_collision_geometry />
-    </collision>
+    <inertial>
+      <!--xacro:left_wheels_inertial_params /-->
+      <origin xyz="0 0 0" rpy="0 0 0"/>
+      <mass value="${tyre_mass}"/>
+      <inertia
+          ixx="${tyre_mass_ixx}"  ixy="0.000000"  ixz="0.000000"
+          iyy="${tyre_mass_iyy}"  iyz="0.000000"
+          izz="${tyre_mass_izz}"/>
+    </inertial>
   </link>
   <joint name="left_front_wheel_joint" type="continuous">
-    <origin xyz="0 0 0" rpy="1.5708 0 0" />
     <parent link="left_steering_hinge" />
     <child link="left_front_wheel" />
-    <axis xyz="0 0 -1" />
-    <limit effort="10" velocity="100" />
-  </joint>
+    <origin xyz="0 ${-str_length/2 - tyre_length/2} 0" rpy="0 0 0"/>
+    <axis xyz="0 1 0" />
+    <dynamics damping="0.1"/>
+    <limit effort="10000" velocity="100" />
+    <joint_properties damping="0.0" friction="0.0" />
+  </joint>
+  <!-- this transmission is added to connect to wheel effort controller! dont delete"-->
   <xacro:wheel_transmission name="left_front_wheel" />
-  <!-- Add the left front wheel with its joints and tranmissions -->
+  <!-- Right Front Wheel -->
   <link name="right_front_wheel">
-    <inertial>
-      <xacro:right_wheels_inertial_params />
-    </inertial>
-    <visual>
-      <xacro:right_front_wheel_geometry />
+    <collision>
+      <!--xacro:right_wheels_collision_geometry /-->
+      <xacro:insert_block name="tyre_origin"/>
+      <geometry>
+        <cylinder length="${tyre_length}" radius="${tyre_radius}"/>
+      </geometry>
+    </collision>
+    <visual>
+      <!--xacro:right_front_wheel_geometry /-->
+      <xacro:insert_block name="tyre_origin"/>
+      <geometry>
+        <cylinder length="${tyre_length}" radius="${tyre_radius}"/>
+      </geometry>
       <material name="black" />
     </visual>
-    <collision>
-      <xacro:right_wheels_collision_geometry />
-    </collision>
+    <inertial>
+      <!--xacro:right_wheels_inertial_params /-->
+      <origin xyz="0 0 0" rpy="0 0 0"/>
+      <mass value="${tyre_mass}"/>
+      <inertia
+          ixx="${tyre_mass_ixx}"  ixy="0.000000"  ixz="0.000000"
+          iyy="${tyre_mass_iyy}"  iyz="0.000000"
+          izz="${tyre_mass_izz}"/>
+    </inertial>
   </link>
   <joint name="right_front_wheel_joint" type="continuous">
-    <origin xyz="0 0 0" rpy="1.5708 0 0" />
     <parent link="right_steering_hinge" />
     <child link="right_front_wheel" />
-    <axis xyz="0 0 -1" />
-    <limit effort="10" velocity="100"/>
-  </joint>
+    <origin xyz="0 ${-str_length/2 - tyre_length/2} 0" rpy="0 0 0"/>
+    <axis xyz="0 1 0" />
+    <dynamics damping="0.1"/>
+    <limit effort="10000" velocity="100" />
+    <joint_properties damping="0.0" friction="0.0" />
+  </joint>
+  <!-- this transmission is added to connect to wheel effort controller! dont delete"-->
   <xacro:wheel_transmission name="right_front_wheel" />
   <!-- Add Hokuyo laser scanner -->
-  <link name="laser">
+  <!--link name="laser">
     <inertial>
       <xacro:hokuyo_inertial_params />
@@ -216,10 +308,10 @@
   <joint name="hokuyo_joint" type="fixed">
     <origin xyz="0.265 0.0 0.075" rpy="0 0 0"/>
-    <parent link="chassis" />
+    <parent link="base_link" />
     <child link="laser" />
     <axis xyz="0 0 1" />
-  </joint>
+  </joint-->
   <!-- zed camera -->
-  <link name="zed_camera_link">
+  <!--link name="zed_camera_link">
     <inertial>
       <mass value="1e-5" />
@@ -243,13 +335,13 @@
   <joint name="zed_camera_joint" type="fixed">
     <origin xyz="0.390 0 0.04" rpy="0 0 0"/>
-    <parent link="chassis"/>
+    <parent link="base_link"/>
     <child link="zed_camera_link"/>
     <axis xyz="0 0 1" />
-    <!-- <limit lower="0.0" upper="0.0" effort="0.0" velocity="0.0" /> -->
-  </joint>
+    <limit lower="0.0" upper="0.0" effort="0.0" velocity="0.0" /-->
+  <!--/joint-->
   <!-- zed camera lenses -->
   <!-- It seems these have to have a non-zero mass to have a camera attached? -->
-  <link name="camera_link"><!-- this needs to match the name in zed_wrapper/zed_tf.launch -->
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
Commit message: looks very promissing

File: src/bobcat_description/urdf/bobcat.xacro (robot description, xacro)
@@ -99,5 +99,5 @@
     <parent link="base_link" />
     <child link="left_rear_wheel" />
-    <origin xyz="${-tyre_x} ${tyre_y} ${tyre_r}" rpy="0 0 0"/>
+    <origin xyz="${-tyre_x} ${tyre_y} ${tyre_r}" rpy="0 0 ${PI}"/>
     <axis xyz="0 1 0" />
     <dynamics damping="0.1"/>
@@ -173,5 +173,5 @@
     <parent link="base_link" />
     <child link="left_steering_hinge" />
-    <origin xyz="${tyre_x} ${car_width/2 + str_length/2} ${tyre_r}" rpy="0 0 0"/>
+    <origin xyz="${tyre_x} ${car_width/2 + str_length/2} ${tyre_r}" rpy="0 0 ${PI}"/>
     <axis xyz="0 0 1"/>
     <limit effort="1000.0" lower="${-str_angle}" upper="${str_angle}" velocity="0.5"/>
@@ -184,5 +184,5 @@
       <xacro:insert_block name="tyre_origin"/>
       <geometry>
-        <cylinder length="${tyre_length}" radius="${tyre_radius}"/>
+        <cylinder length="${str_length}" radius="${str_radius}"/>
       </geometry>
     </collision>

Commit message: BAM ackermann vehicle working quite nice! whats left to do is add the lidar and camera back to the vehicle and then create some meshes, try weights for actual racecar and yea

File: src/bobcat_description/urdf/bobcat.xacro (robot description, xacro)
@@ -100,7 +100,7 @@
     <child link="left_rear_wheel" />
     <origin xyz="${-tyre_x} ${tyre_y} ${tyre_r}" rpy="0 0 ${PI}"/>
-    <axis xyz="0 1 0" />
+    <axis xyz="0 -1 0" />
     <dynamics damping="0.1"/>
-    <limit effort="10000" velocity="100" />
+    <limit effort="100000" velocity="1000" />
     <joint_properties damping="0.0" friction="0.0" />
   </joint>
@@ -140,5 +140,5 @@
     <axis xyz="0 1 0"/>
     <dynamics damping="0.1"/>
-    <limit effort="10000" velocity="100" />
+    <limit effort="100000" velocity="1000" />
     <joint_properties damping="0.0" friction="0.0" />
   </joint>
