Commit message: 6h later i'd say the result is quite promising, testet most of it and it should be at least so good that one can work with it

File: src/bobcat_description/urdf/bobcat.xacro (robot description, xacro)
@@ -99,4 +99,5 @@
     <parent link="base_link" />
     <child link="left_rear_wheel" />
+<!-- here y is PI as the car will be mounted in the same direction as the right wheel and that somewhat seems wrong. When you turn this back for whatever reason remember to set axis to +1 as it will turn in the wrong direction otherwise -->
     <origin xyz="${-tyre_x} ${tyre_y} ${tyre_r}" rpy="0 0 ${PI}"/>
     <axis xyz="0 -1 0" />
@@ -288,5 +289,5 @@
   <xacro:wheel_transmission name="right_front_wheel" />
   <!-- Add Hokuyo laser scanner -->
-  <!--link name="laser">
+  <link name="laser">
     <inertial>
       <xacro:hokuyo_inertial_params />
@@ -307,11 +308,11 @@
   </link>
   <joint name="hokuyo_joint" type="fixed">
-    <origin xyz="0.265 0.0 0.075" rpy="0 0 0"/>
+    <origin xyz="${tyre_x - 0.1} 0 ${car_height + tyre_r + 0.05}" />
     <parent link="base_link" />
     <child link="laser" />
     <axis xyz="0 0 1" />
-  </joint-->
+  </joint>
   <!-- zed camera -->
-  <!--link name="zed_camera_link">
+  <link name="zed_camera_link">
     <inertial>
       <mass value="1e-5" />
@@ -334,14 +335,14 @@
   </link>
   <joint name="zed_camera_joint" type="fixed">
-    <origin xyz="0.390 0 0.04" rpy="0 0 0"/>
+     <origin xyz="${tyre_x + 0.016} 0 ${car_height + tyre_r/2 }" />
     <parent link="base_link"/>
     <child link="zed_camera_link"/>
     <axis xyz="0 0 1" />
-    <limit lower="0.0" upper="0.0" effort="0.0" velocity="0.0" /-->
-  <!--/joint-->
+    <!--limit lower="0.0" upper="0.0" effort="0.0" velocity="0.0" /-->
+  </joint>
   <!-- zed camera lenses -->
   <!-- It seems these have to have a non-zero mass to have a camera attached? -->
-  <!--link name="camera_link"--><!-- this needs to match the name in zed_wrapper/zed_tf.launch -->
-    <!--inertial>
+  <link name="camera_link"><!-- this needs to match the name in zed_wrapper/zed_tf.launch -->
+    <inertial>
       <mass value="1e-5" />
       <origin xyz="0 0 0" rpy="0 0 0"/>
@@ -367,5 +368,5 @@
     <child link="zed_camera_right_link"/>
     <axis xyz="0 0 1" />
-  </joint-->
+  </joint>
   <!-- Add the remaining xacros -->
   <xacro:include filename="$(find bobcat_description)/urdf/bobcat.gazebo" />

Commit message: error in ackermann.py that calculated wrong speed fixed. simulation environment now in a state that one can use it pretty comfortable

File: src/bobcat_description/urdf/bobcat.xacro (robot description, xacro)
@@ -4,27 +4,27 @@
   <xacro:property name="PI" value="3.1415926835897931"/>
 <!--  <xacro:property name="base_height" value="0"/> -->
-  <xacro:property name="base_height" value="1.0639"/>
-  <xacro:property name="base_mass" value="2050"/>
-  <xacro:property name="base_mass_ixx" value="63"/>
-  <xacro:property name="base_mass_iyy" value="1048"/>
-  <xacro:property name="base_mass_izz" value="1111"/>
-  <xacro:property name="base_mass_ixz" value="-31"/>
-  <xacro:property name="tyre_x" value="1.31"/>
-  <xacro:property name="tyre_y" value="0.765"/>
+  <xacro:property name="base_height" value="0.4"/>
+  <xacro:property name="base_mass" value="1000"/>
+  <xacro:property name="base_mass_ixx" value="30"/>
+  <xacro:property name="base_mass_iyy" value="500"/>
+  <xacro:property name="base_mass_izz" value="550"/>
+  <xacro:property name="base_mass_ixz" value="-15"/>
+  <xacro:property name="tyre_x" value="0.76"/>
+  <xacro:property name="tyre_y" value="0.5"/>
   <xacro:property name="tyre_length" value="0.229"/>
   <xacro:property name="tyre_height" value="-0.696"/>
-  <xacro:property name="tyre_r" value="0.66"/>
-  <xacro:property name="tyre_radius" value="0.356"/>
-  <xacro:property name="tyre_mass" value="40"/>
-  <xacro:property name="tyre_mass_ixx" value="54"/>
-  <xacro:property name="tyre_mass_iyy" value="56"/>
-  <xacro:property name="tyre_mass_izz" value="104"/>
-  <xacro:property name="car_height" value="0.8"/>
-  <xacro:property name="car_width" value="1.301"/>
-  <xacro:property name="car_length" value="2.62"/>
+  <xacro:property name="tyre_r" value="0.22"/>
+  <xacro:property name="tyre_radius" value="0.22"/>
+  <xacro:property name="tyre_mass" value="3"/>
+  <xacro:property name="tyre_mass_ixx" value="20"/>
+  <xacro:property name="tyre_mass_iyy" value="20"/>
+  <xacro:property name="tyre_mass_izz" value="50"/>
+  <xacro:property name="car_height" value="0.6"/>
+  <xacro:property name="car_width" value="1.0"/>
+  <xacro:property name="car_length" value="1.54"/>
   <xacro:property name="camera_box" value="0.1"/>
   <xacro:property name="str_length" value="0.01"/>
   <xacro:property name="str_radius" value="0.1"/>
-  <xacro:property name="str_angle" value="0.6"/>
+  <xacro:property name="str_angle" value="0.5"/>
   <xacro:property name="tyre_origin">
 	<origin xyz="0 0 0" rpy="${PI/2} 0 0"/>
@@ -48,4 +48,5 @@
       <origin xyz="0 0 ${base_height}" rpy="0 0 0" />
       <geometry>
+	 <!--mesh><uri>file://kappa_scene.dae</uri></mesh-->
         <box size="${car_length} ${car_width} ${car_height}"/>
       </geometry>
@@ -63,4 +64,5 @@
           izz="${base_mass_izz}"/>
       </inertial>
+      <dampingFactor>0.1</dampingFactor>
   </link>
   <joint name="inertia_joint" type="fixed">
@@ -100,8 +102,8 @@
     <child link="left_rear_wheel" />
 <!-- here y is PI as the car will be mounted in the same direction as the right wheel and that somewhat seems wrong. When you turn this back for whatever reason remember to set axis to +1 as it will turn in the wrong direction otherwise -->
-    <origin xyz="${-tyre_x} ${tyre_y} ${tyre_r}" rpy="0 0 ${PI}"/>
+    <origin xyz="${-tyre_x} ${car_width/2 + tyre_length/2} ${tyre_r}" rpy="0 0 ${PI}"/>
     <axis xyz="0 -1 0" />
-    <dynamics damping="0.1"/>
-    <limit effort="100000" velocity="1000" />
+    <dynamics damping="0.2"/>
+    <limit effort="100000" velocity="100" />
     <joint_properties damping="0.0" friction="0.0" />
   </joint>
@@ -138,8 +140,8 @@
     <parent link="base_link" />
     <child link="right_rear_wheel" />
-    <origin xyz="${-tyre_x} ${-tyre_y} ${tyre_r}" rpy="0 0 0"/>
+    <origin xyz="${-tyre_x} ${-car_width/2 - tyre_length/2} ${tyre_r}" rpy="0 0 0"/>
     <axis xyz="0 1 0"/>
-    <dynamics damping="0.1"/>
-    <limit effort="100000" velocity="1000" />
+    <dynamics damping="0.2"/>
+    <limit effort="100000" velocity="100" />
     <joint_properties damping="0.0" friction="0.0" />
   </joint>
@@ -176,5 +178,5 @@
     <origin xyz="${tyre_x} ${car_width/2 + str_length/2} ${tyre_r}" rpy="0 0 ${PI}"/>
     <axis xyz="0 0 1"/>
-    <limit effort="1000.0" lower="${-str_angle}" upper="${str_angle}" velocity="0.5"/>
+    <limit effort="1000.0" lower="${-str_angle}" upper="${str_angle}" velocity="1.0"/>
   </joint>
   <!-- this transmission is added to connect to wheel effort controller! dont delete"-->
@@ -208,5 +210,5 @@
     <origin xyz="${tyre_x} ${-car_width/2 - str_length/2} ${tyre_r}" rpy="0 0 0"/>
     <axis xyz="0 0 1"/>
-    <limit effort="1000.0" lower="${-str_angle}" upper="${str_angle}" velocity="0.5"/>
+    <limit effort="1000.0" lower="${-str_angle}" upper="${str_angle}" velocity="1.0"/>
   </joint>
   <!-- this transmission is added to connect to wheel effort controller! dont delete"-->
@@ -308,5 +310,5 @@
   </link>
   <joint name="hokuyo_joint" type="fixed">
-    <origin xyz="${tyre_x - 0.1} 0 ${car_height + tyre_r + 0.05}" />
+    <origin xyz="${tyre_x + 0.1} 0 ${car_height - tyre_r/2}" />
     <parent link="base_link" />
     <child link="laser" />
@@ -335,5 +337,5 @@
   </link>
   <joint name="zed_camera_joint" type="fixed">
-     <origin xyz="${tyre_x + 0.016} 0 ${car_height + tyre_r/2 }" />
+    <origin xyz="${tyre_x} 0 ${car_height + tyre_r/2}" />
     <parent link="base_link"/>
     <child link="zed_camera_link"/>

Commit message: repaired the world file and added odom and imu also added extended kalman filter that is not using gps for now (someone could integrate it) also got the gmapping node running! we might want to retry the lidar test we did at the faps derpartment with this package to see how good the lidar really is

File: src/bobcat_description/urdf/bobcat.xacro (robot description, xacro)
@@ -290,4 +290,30 @@
   <!-- this transmission is added to connect to wheel effort controller! dont delete"-->
   <xacro:wheel_transmission name="right_front_wheel" />
+<!-- Add IMU -->
+<link name="imu_link">
+  <inertial>
+    <mass value="0.001"/>
+    <origin rpy="0 0 0" xyz="0 0 0"/>
+    <inertia ixx="0.0001" ixy="0" ixz="0" iyy="0.000001" iyz="0" izz="0.0001"/>
+  </inertial>
+  <visual>
+    <origin rpy="0 0 0" xyz="0 0 0"/>
+    <geometry>
+      <box size="0.001 0.001 0.001"/>
+    </geometry>
+  </visual>
+  <collision>
+    <origin rpy="0 0 0" xyz="0 0 0"/>
+    <geometry>
+      <box size=".001 .001 .001"/>
+    </geometry>
+  </collision>
+</link>
+  <joint name="imu_joint" type="fixed">
+    <axis xyz="1 0 0"/> <!-- 0 1 0 -->
+    <origin xyz="0 0 0.19"/>
+    <parent link="base_link"/>
+    <child link="imu_link"/>
+  </joint>
   <!-- Add Hokuyo laser scanner -->
   <link name="laser">

Commit message: detect impuls updated to higher pwm

File: src/bobcat_description/urdf/bobcat.xacro (robot description, xacro)
@@ -336,5 +336,6 @@
   </link>
   <joint name="hokuyo_joint" type="fixed">
-    <origin xyz="${tyre_x + 0.1} 0 ${car_height - tyre_r/2}" />
+    <!--origin xyz="${tyre_x + 0.1} 0 ${car_height - tyre_r/2}" /-->
+    <origin xyz="${tyre_x + 0.1} 0 0.2" />
     <parent link="base_link" />
     <child link="laser" />
